Commit message: finish rviz && gazebo test

File: catkin_ws/src/wpb_home/wpb_home_bringup/urdf/wpb_home.urdf (robot description, URDF)
Before this commit: robot wpb_home, 7 links, 6 joints
Joints:
- joint kinect_height: origin xyz=0.000 -0.100 0 rpy=0 -1.5707963 0 -> xyz=0.170 -0.100 0 rpy=0 -1.5707963 0

Commit message: 优化前端逻辑，通过前端启动仿真/连接实机，并且启用相关节点。启动前可以配置参数。

File: catkin_ws/src/wpb_home/wpb_home_bringup/urdf/wpb_home.urdf (robot description, URDF)
Before this commit: robot wpb_home, 7 links, 6 joints
Joints:
- joint kinect_height: origin xyz=0.170 -0.100 0 rpy=0 -1.5707963 0 -> xyz=${wpb_config['camera_mount']['x']} ${wpb_config['camera_mount']['y']} ${wpb_config['camera_mount']['z']} rpy=0 -1.5707963 0
